File: Schematics/ESP32_Shield/ESP32_Shield/ESP32_Shield.kicad_pcb (KiCad board)
At the start: 2 copper layers, 26.2 x 49.5 mm, 18 parts, among them J1 Conn_01x10, Q3 Si2319CDS, Q4 Si2319CDS, U6 ADS1234IPW, U7 SHT30-DIS

Commit message: Order ready
Parts:
- added R22: 100k, Resistor_SMD:R_0603_1608Metric_Pad0.98x0.95mm_HandSolder, F.Cu at (116.0, 91.5)
- R14, R15: value 510k -> 100k
- R21: value 10k -> 100k
- moved C13 12.7 mm to (127.1, 101.1)
- moved C12 9.85 mm to (124.0, 90.3), turned to 0 degrees
- moved R18 5.54 mm to (128.0, 73.9), turned to 180 degrees
- moved U6 2.10 mm to (125.4, 95.2), turned to -90 degrees
- moved R13 1.35 mm to (128.0, 71.0), turned to 180 degrees
- moved Q4 1.15 mm to (116.9, 95.6), turned to -90 degrees
Connections:
- C14 pad 1: GND -> -BATT
- Q3 pad 2: Net-(Q3-S) -> +BATT
- Q3 pad 3: +BATT -> Net-(Q3-D)
- R14 pad 1: Net-(Q3-S) -> Net-(Q3-D)
- R15 pad 1: GND -> -BATT
- U2 pad 2: !EN_DMS -> unconnected-(U2-IO36-Pad2)
- U2 pad 22: unconnected-(U2-IO17-Pad22) -> !EN_DMS
- U2 pad 23: unconnected-(U2-IO5-Pad23) -> !en_meas
- U2 pad 24: SCLK -> unconnected-(U2-IO18-Pad24)
- U2 pad 3: !en_meas -> unconnected-(U2-IO39-Pad3)
Routing:
- net +3.3V: track 0.00 -> 66.6 mm, vias 0 -> 8
- net -BATT: track 0.00 -> 53.5 mm, vias 0 -> 4
- net +BATT: track 0.00 -> 51.2 mm
- net Net-(J1-Pin_2): track 0.00 -> 39.3 mm, vias 0 -> 2
- net !en_meas: track 0.00 -> 37.9 mm
- net Net-(J1-Pin_9): track 0.00 -> 31.8 mm, vias 0 -> 2
- net Net-(J1-Pin_10): track 0.00 -> 31.5 mm, vias 0 -> 4
- net !PWDN: track 0.00 -> 30.0 mm, vias 0 -> 2
- net GND: track 0.00 -> 29.8 mm, vias 0 -> 18
- net SCL: track 0.00 -> 27.7 mm
- net !EN_DMS: track 0.00 -> 25.3 mm, vias 0 -> 4
- net SDA: track 0.00 -> 17.7 mm, vias 0 -> 2
- net Net-(J1-Pin_5): track 0.00 -> 15.5 mm, vias 0 -> 2
- net bat_adc: track 0.00 -> 15.3 mm
- net Net-(J1-Pin_6): track 0.00 -> 14.0 mm, vias 0 -> 2
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- added copper zone on B.Cu, net GND
Other:
- board size 26.2 x 49.5 mm -> 26.6 x 50.4 mm

Commit message: korrekturen
Parts:
- removed Q3: Si2319CDS, Package_TO_SOT_SMD:SOT-23
- removed R21: 100k, Resistor_SMD:R_0603_1608Metric_Pad0.98x0.95mm_HandSolder
- added C1: 0.1u, Capacitor_SMD:C_0603_1608Metric_Pad1.08x0.95mm_HandSolder, F.Cu at (128.2, 101.0)
- added Q1: Si1308EDL, Package_TO_SOT_SMD:SOT-323_SC-70, F.Cu at (118.2, 80.0)
- moved C13 2.60 mm to (124.5, 101.0)
Connections:
- BAT_VOLT1 pad 1: -BATT -> +BATT
- BAT_VOLT1 pad 2: +BATT -> GND
- C14 pad 1: -BATT -> GND
- C14 pad 2: bat_adc -> en_meas
- R14 pad 1: Net-(Q3-D) -> +BATT
- R15 pad 1: -BATT -> Net-(Q1-D)
- U2 pad 23: !en_meas -> en_meas
Routing:
- net +3.3V: track 66.6 -> 190.4 mm, vias 8 -> 3
- net -BATT: track 53.5 -> 0.00 mm, vias 4 -> 0
- net !en_meas: track 37.9 -> 0.00 mm
- net en_meas: track 0.00 -> 25.7 mm, vias 0 -> 2
- net Net-(J1-Pin_2): track 39.3 -> 24.8 mm
- net Net-(Q3-D): track 8.33 -> 0.00 mm
- net Net-(J1-Pin_5): track 15.5 -> 22.8 mm, vias 2 -> 0
- net Net-(Q1-D): track 0.00 -> 6.14 mm
- net +BATT: track 51.2 -> 54.9 mm
- net bat_adc: track 15.3 -> 13.2 mm
- net Net-(J1-Pin_8): track 11.9 -> 13.3 mm
- net Net-(J1-Pin_7): track 10.2 -> 11.0 mm
- net SCLK: track 9.11 -> 9.51 mm, vias 2 -> 1
- net !EN_DMS: track 25.3 -> 25.0 mm, vias 4 -> 3
- net D_RDY_OUT: track 9.52 -> 9.67 mm, vias 2 -> 1
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Other:
- board size 26.6 x 50.4 mm -> 27 x 50.2 mm

Commit message: ...
Parts:
- moved R15 2.09 mm to (119.0, 83.6), turned to -90 degrees
- moved Q1 0.71 mm to (117.8, 79.5), turned to -90 degrees
- moved C14 0.66 mm to (121.8, 85.8)
- moved R14 0.15 mm to (117.3, 83.6), turned to -90 degrees
Routing:
- net Net-(Q1-D): track 6.14 -> 2.77 mm
- net bat_adc: track 13.2 -> 12.2 mm
- net +BATT: track 54.9 -> 54.2 mm
- net !PWDN: vias 2 -> 1

Commit message: Feedback umetzen
Parts:
- added ADC1: Conn_01x02, Connector_PinHeader_2.54mm:PinHeader_1x02_P2.54mm_Vertical, F.Cu at (128.8, 86.7)
- added DMS1: Conn_01x02, Connector_PinHeader_2.54mm:PinHeader_1x02_P2.54mm_Vertical, F.Cu at (135.3, 116.0)
- added ESP32: Conn_01x02, Connector_PinHeader_2.54mm:PinHeader_1x02_P2.54mm_Vertical, F.Cu at (123.0, 110.0)
- added Q3: Si2319CDS, Package_TO_SOT_SMD:SOT-23, F.Cu at (118.2, 71.2)
- added R21: 100k, Resistor_SMD:R_0603_1608Metric_Pad0.98x0.95mm_HandSolder, F.Cu at (118.2, 75.5)
- added THRM1: Conn_01x02, Connector_PinHeader_2.54mm:PinHeader_1x02_P2.54mm_Vertical, F.Cu at (124.5, 66.7)
- Q1: footprint Package_TO_SOT_SMD:SOT-323_SC-70 -> Package_TO_SOT_SMD:SOT-23
- moved V_IN1 11.1 mm to (112.7, 116.0)
- moved C1 10.9 mm to (129.1, 90.1), turned to 0 degrees
- moved U7 10.1 mm to (123.1, 72.5), turned to 180 degrees
- moved C14 2.86 mm to (123.5, 83.5), turned to -90 degrees
- moved PWR1 2.83 mm to (112.7, 110.0), turned to 90 degrees
- moved C13 2.11 mm to (126.4, 100.1), turned to 180 degrees
- moved R15 1.50 mm to (120.5, 83.6)
- moved C12 0.92 mm to (123.8, 89.4)
- moved Q1 0.90 mm to (118.2, 78.8), turned to 90 degrees
- moved BAT1 0.57 mm to (132.2, 110.0)
- renumbered BAT_VOLT1 to BAT1, PWR_MON1 to PWR1, PWR1 to V_IN1
Connections:
- C1 pad 2: +3.3V -> Net-(ADC1-Pin_2)
- C13 pad 2: Net-(J1-Pin_2) -> Net-(ADC1-Pin_2)
- C14 pad 2: en_meas -> bat_adc
- C15 pad 1: +3.3V -> Net-(THRM1-Pin_2)
- Q4 pad 2: +3.3V -> Net-(DMS1-Pin_2)
- R14 pad 1: +BATT -> Net-(Q3-D)
- R15 pad 1: Net-(Q1-D) -> GND
- R22 pad 2: +3.3V -> Net-(DMS1-Pin_2)
- U2 pad 15: +5V -> Net-(ESP32-Pin_2)
- U6 pad 1: +3.3V -> Net-(ADC1-Pin_2)
- U6 pad 20: Net-(J1-Pin_2) -> Net-(ADC1-Pin_2)
- U6 pad 22: Net-(J1-Pin_2) -> Net-(ADC1-Pin_2)
- U6 pad 23: +3.3V -> Net-(ADC1-Pin_2)
- U6 pad 24: +3.3V -> Net-(ADC1-Pin_2)
- U7 pad 5: +3.3V -> Net-(THRM1-Pin_2)
Routing:
- net +3.3V: track 190.1 -> 73.8 mm, vias 3 -> 4
- net Net-(DMS1-Pin_2): track 0.00 -> 38.8 mm
- net Net-(ADC1-Pin_2): track 0.00 -> 36.4 mm, vias 0 -> 2
- net Net-(ESP32-Pin_2): track 0.00 -> 23.0 mm
- net Net-(THRM1-Pin_2): track 0.00 -> 18.2 mm
- net Net-(J1-Pin_2): track 24.8 -> 9.31 mm, vias 2 -> 0
- net Net-(Q3-D): track 0.00 -> 15.1 mm
- net SCL: track 27.7 -> 14.3 mm
- net bat_adc: track 12.2 -> 24.5 mm
- net Net-(J1-Pin_9): track 31.8 -> 24.5 mm
- net Net-(J1-Pin_10): track 31.5 -> 24.5 mm, vias 4 -> 2
- net Net-(J1-Pin_5): track 22.8 -> 16.5 mm, vias 0 -> 1
- net en_meas: track 25.7 -> 19.6 mm, vias 2 -> 0
- net SDA: track 17.7 -> 12.5 mm, vias 2 -> 0
- net !PWDN: track 30.0 -> 25.6 mm, vias 1 -> 0
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- added copper zone on F.Cu, net GND
Other:
- board size 27 x 50.2 mm -> 27.4 x 55.8 mm
- board text added: "Thomas Rocheteau BA26_brnn_241"

Commit message: a
Parts:
- added C6: 10u, Capacitor_SMD:C_0603_1608Metric_Pad1.08x0.95mm_HandSolder, F.Cu at (119.8, 114.3)
- added C7: 22u, Capacitor_SMD:C_0603_1608Metric_Pad1.08x0.95mm_HandSolder, F.Cu at (127.0, 120.1)
- added ESP3.3V1: Conn_01x02, Connector_PinHeader_2.54mm:PinHeader_1x02_P2.54mm_Vertical, F.Cu at (135.3, 121.5)
- added L1: 0.47u, Inductor_SMD:L_Coilcraft_XxL4020, F.Cu at (128.3, 115.9)
- added R8: 511k, Resistor_SMD:R_0603_1608Metric_Pad0.98x0.95mm_HandSolder, F.Cu at (122.5, 120.1)
- added R9: 91k, Resistor_SMD:R_0603_1608Metric_Pad0.98x0.95mm_HandSolder, F.Cu at (119.5, 117.4)
- added S1: JS202011SCQN, Button_Switch_SMD:SW_DPDT_CK_JS202011JCQN, F.Cu at (115.5, 122.6)
- added U4: TPS63802DLAR, TPS63802DLAR:VREG_TPS63802DLAR, F.Cu at (123.2, 116.3)
- renumbered V_IN1 to 6V_IN1, ESP32 to ESP5V1
Connections:
- ESP5V1 pad 1: +5V -> 5V LDO
- U2 pad 16: +3.3V -> Net-(ESP3.3V1-Pin_2)
Routing:
- net +3.3V: track 73.8 -> 96.9 mm, vias 4 -> 5
- net Net-(ESP3.3V1-Pin_2): track 0.00 -> 22.7 mm, vias 0 -> 2
- net 5V LDO: track 0.00 -> 16.9 mm, vias 0 -> 1
- net 5V BUCK: track 0.00 -> 16.7 mm
- net Net-(U4-FB): track 0.00 -> 5.37 mm
- net +5V: track 8.00 -> 12.8 mm
- net Net-(U4-L1): track 0.00 -> 4.75 mm
- net Net-(U4-L2): track 0.00 -> 4.42 mm
- net GND: track 28.1 -> 26.6 mm
Other:
- board size 27.4 x 55.8 mm -> 27.3 x 62.9 mm

Commit message: a
Other:
- board text added: "D15"
- board text added: "D2"
- board text added: "D4"
- board text added: "RX2"
- board text added: "TX2, IO17"
Changed lines of the file:
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@@
+		)
+	)
+	(gr_text "RX2"
+		(at 138.2 88.35 0)
+		(layer "User.1")
+		(effects
+			(font
+				(size 1.5 1.5)
+				(thickness 0.3)
+				(bold yes)
+			)
+			(justify left bottom)
+		)
+	)
+	(gr_text "TX2, IO17"
+		(at 138.25 86.15 0)
+		(layer "User.1")
+		(effects
+			(font
+				(size 1.5 1.5)
+				(thickness 0.3)
+				(bold yes)
+			)
+			(justify left bottom)
+		)
+	)
+	(gr_text "D4"
+		(at 138.2 90.85 0)
+		(layer "User.1")
+		(effects
+			(font
+				(size 1.5 1.5)
+				(thickness 0.3)
+				(bold yes)
+			)
+			(justify left bottom)
+		)
+	)
+	(gr_text "D2"
+		(at 138.3 93.5 0)
+		(layer "User.1")
+		(effects
+			(font
+				(size 1.5 1.5)
+				(thickness 0.3)
+				(bold yes)
+			)
+			(justify left bottom)
+		)
+	)
+	(gr_text "D15"
+		(at 138.2 96.35 0)
+		(layer "User.1")
+		(effects
+			(font
+				(size 1.5 1.5)
+				(thickness 0.3)
+				(bold yes)
+			)
+			(justify left bottom)
 		)
 	)
