File: Schematics/ESP32_Shield 2/ESP32_Shield 2.kicad_pcb (KiCad board)
At the start: 2 copper layers, 27.3 x 62.9 mm, 34 parts, among them IC1 TPS62842DGRR, J1 Conn_01x10, Q1 Si1308EDL, Q3 Si2319CDS, Q4 Si2319CDS, U4 TPS63802DLAR, U6 ADS1234IPW, U7 SHT30-DIS

Commit message: k
Parts:
- removed C6: 10u, Capacitor_SMD:C_0603_1608Metric_Pad1.08x0.95mm_HandSolder
- removed C7: 22u, Capacitor_SMD:C_0603_1608Metric_Pad1.08x0.95mm_HandSolder
- removed IC1: TPS62842DGRR, SamacSys_Parts:SOP65P490X110-9N
- removed R8: 511k, Resistor_SMD:R_0603_1608Metric_Pad0.98x0.95mm_HandSolder
- removed R9: 91k, Resistor_SMD:R_0603_1608Metric_Pad0.98x0.95mm_HandSolder
- removed U4: TPS63802DLAR, TPS63802DLAR:VREG_TPS63802DLAR
- added C16: 10u, Capacitor_SMD:C_0603_1608Metric_Pad1.08x0.95mm_HandSolder, F.Cu at (120.9, 123.2)
- added C17: 4.7u, Capacitor_SMD:C_0603_1608Metric_Pad1.08x0.95mm_HandSolder, F.Cu at (127.5, 129.8)
- added C18: 1u, Capacitor_SMD:C_0603_1608Metric_Pad1.08x0.95mm_HandSolder, F.Cu at (118.4, 107.9)
- added C19: 10n, Capacitor_SMD:C_0603_1608Metric_Pad1.08x0.95mm_HandSolder, F.Cu at (121.2, 106.9)
- added C20: 10n, Capacitor_SMD:C_0603_1608Metric_Pad1.08x0.95mm_HandSolder, F.Cu at (118.4, 105.8)
- added C21: 1u, Capacitor_SMD:C_0603_1608Metric_Pad1.08x0.95mm_HandSolder, F.Cu at (124.0, 107.9)
- added C22: 10n, Capacitor_SMD:C_0603_1608Metric_Pad1.08x0.95mm_HandSolder, F.Cu at (126.7, 106.8)
- added C23: 10n, Capacitor_SMD:C_0603_1608Metric_Pad1.08x0.95mm_HandSolder, F.Cu at (124.0, 105.8)
- added C24: 1u, Capacitor_SMD:C_0603_1608Metric_Pad1.08x0.95mm_HandSolder, F.Cu at (129.4, 107.9)
- added C25: 10n, Capacitor_SMD:C_0603_1608Metric_Pad1.08x0.95mm_HandSolder, F.Cu at (132.2, 106.8)
- added C26: 10n, Capacitor_SMD:C_0603_1608Metric_Pad1.08x0.95mm_HandSolder, F.Cu at (129.4, 105.8)
- added C27: 1u, Capacitor_SMD:C_0603_1608Metric_Pad1.08x0.95mm_HandSolder, F.Cu at (135.0, 107.9)
- added C28: 10n, Capacitor_SMD:C_0603_1608Metric_Pad1.08x0.95mm_HandSolder, F.Cu at (137.6, 106.8)
- added C29: 10n, Capacitor_SMD:C_0603_1608Metric_Pad1.08x0.95mm_HandSolder, F.Cu at (134.9, 105.8)
- added IC2: TPS62842DGRR, SamacSys_Parts:SOP65P490X110-9N, F.Cu at (124.0, 126.9)
- added R16: 52.3k, Resistor_SMD:R_0603_1608Metric_Pad0.98x0.95mm_HandSolder, F.Cu at (122.5, 129.7)
- added R17: 100, Resistor_SMD:R_0603_1608Metric_Pad0.98x0.95mm_HandSolder, F.Cu at (117.6, 111.0)
- added R19: 100, Resistor_SMD:R_0603_1608Metric_Pad0.98x0.95mm_HandSolder, F.Cu at (120.2, 111.0)
- added R20: 100, Resistor_SMD:R_0603_1608Metric_Pad0.98x0.95mm_HandSolder, F.Cu at (125.3, 111.0)
- added R23: 100, Resistor_SMD:R_0603_1608Metric_Pad0.98x0.95mm_HandSolder, F.Cu at (122.8, 111.0)
- added R24: 100, Resistor_SMD:R_0603_1608Metric_Pad0.98x0.95mm_HandSolder, F.Cu at (130.3, 111.0)
- added R25: 100, Resistor_SMD:R_0603_1608Metric_Pad0.98x0.95mm_HandSolder, F.Cu at (127.8, 111.0)
- added R26: 100, Resistor_SMD:R_0603_1608Metric_Pad0.98x0.95mm_HandSolder, F.Cu at (135.4, 111.0)
- added R27: 100, Resistor_SMD:R_0603_1608Metric_Pad0.98x0.95mm_HandSolder, F.Cu at (132.9, 111.0)
- L1: value 0.47u -> 2.2u; footprint Inductor_SMD:L_Coilcraft_XxL4020 -> Capacitor_SMD:C_0805_2012Metric_Pad1.18x1.45mm_HandSolder
- moved L1 13.7 mm to (119.2, 126.1)
- moved J1 10.5 mm to (112.6, 115.0)
- moved S1 9.68 mm to (115.5, 132.3)
- moved 6V_IN1 9.67 mm to (112.7, 125.7)
- moved BAT1 9.67 mm to (132.2, 119.7)
- moved DMS1 9.67 mm to (135.3, 125.7)
- moved ESP3.3V1 9.67 mm to (135.3, 131.2)
- moved ESP5V1 9.67 mm to (123.0, 119.7)
- moved PWR1 9.67 mm to (112.7, 119.7)
Connections:
- L1 pad 1: Net-(U4-L1) -> 3v3 BUCK
- S1 pad 4: unconnected-(S1-Pad4) -> Net-(ESP3.3V1-Pin_2)
- S1 pad 5: unconnected-(S1-Pad5) -> +3.3V
- S1 pad 6: unconnected-(S1-Pad6) -> 3v3 BUCK
- U2 pad 19: D_RDY_OUT -> A1
- U2 pad 29: unconnected-(U2-IO23-Pad29) -> SCL
- U2 pad 7: A1 -> D_RDY_OUT
- U6 pad 11: Net-(J1-Pin_10) -> Net-(U6-AINP1)
- U6 pad 12: Net-(J1-Pin_9) -> Net-(U6-AINN1)
- U6 pad 13: Net-(J1-Pin_6) -> P3
- U6 pad 14: Net-(J1-Pin_5) -> N3
- U6 pad 15: Net-(J1-Pin_3) -> N4
- U6 pad 16: Net-(J1-Pin_4) -> P4
- U6 pad 17: Net-(J1-Pin_7) -> N2
- U6 pad 18: Net-(J1-Pin_8) -> P2
- U6 pad 7: GND -> A1
- U6 pad 8: GND -> A0
Routing:
- net Net-(U6-AINP1): track 0.00 -> 34.3 mm, vias 0 -> 2
- net Net-(ESP3.3V1-Pin_2): track 22.7 -> 56.9 mm
- net Net-(U6-AINN1): track 0.00 -> 33.3 mm, vias 0 -> 2
- net D_RDY_OUT: track 8.03 -> 36.5 mm, vias 0 -> 3
- net P3: track 0.00 -> 24.9 mm, vias 0 -> 2
- net A1: track 0.00 -> 24.5 mm
- net N3: track 0.00 -> 24.0 mm, vias 0 -> 2
- net A0: track 0.00 -> 23.5 mm
- net Net-(J1-Pin_10): track 24.5 -> 3.10 mm, vias 2 -> 0
- net Net-(J1-Pin_9): track 24.5 -> 3.09 mm, vias 2 -> 0
- net P2: track 0.00 -> 20.6 mm
- net N2: track 0.00 -> 18.6 mm
- net +3.3V: track 96.9 -> 113.8 mm
- net N4: track 0.00 -> 16.2 mm
- net 3v3 BUCK: track 0.00 -> 15.8 mm, vias 0 -> 2
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- added copper zone on F.Cu, net 3v3 BUCK
Other:
- board size 27.3 x 62.9 mm -> 30.1 x 74.2 mm
- board text removed: "D15"
- board text removed: "D2"
- board text removed: "D4"
- board text removed: "RX2"
- board text removed: "TX2, IO17"
