File: Schematics/ESP32_Shield 2/ESP32_Shield 2.kicad_sch (KiCad schematic)
At the start: 32 parts, among them IC1 TPS62842DGRR, J1 Conn_01x10, Q1 Si1308EDL, Q3 Si2319CDS, Q4 Si2319CDS, U6 ADS1234IPW, U7 SHT30-DIS

Commit message: k
Parts:
- removed IC1: TPS62842DGRR, SOP65P490X110-9N, symbol SamacSys_Parts:TPS62842DGRR
- added C18, C21, C24, C27: 1u, Capacitor_SMD:C_0603_1608Metric_Pad1.08x0.95mm_HandSolder, symbol Device:C
- added C19, C20, C22, C23, C25, C26, C28, C29: 10n, Capacitor_SMD:C_0603_1608Metric_Pad1.08x0.95mm_HandSolder, symbol Device:C
- added IC2: TPS62842DGRR, SOP65P490X110-9N, symbol SamacSys_Parts:TPS62842DGRR
- added R17, R19, R20, R23, R24, R25, R26, R27: 100, Resistor_SMD:R_0603_1608Metric_Pad0.98x0.95mm_HandSolder, symbol Device:R
- L1: footprint (none) -> Capacitor_SMD:C_0805_2012Metric_Pad1.18x1.45mm_HandSolder
Connections:
- net +3.3V: now also S1.5
- net 5V BUCK: now also IC2.3 (MODE), IC2.5 (EN), IC2.6 (VIN)
- net A0: now also U2.20 (IO4); no longer U2.7 (IO32)
- net A1: now also U2.19 (IO2); no longer U2.20 (IO4)
- net D_RDY_OUT: now also U2.7 (IO32); no longer U2.19 (IO2)
- net GND: now also C19.1, C20.1, C22.1, C23.1, C25.1, C26.1, C28.1, C29.1, IC2.8 (GND_1), IC2.9 (GND_2)
- net SCL: now also U2.29 (IO23)
- net 3v3 BUCK: now reaches C16.2, L1.1
- net 3v3 BUCK: now also S1.6, IC2.1 (VOS)
- net at L1.2: now also IC2.2 (SW)
- net at R16.1: now also IC2.4 (VSET)
- net at U6.11 (AINP1): now also C27.2, C28.2, R26.2; no longer J1.10 (Pin_10)
- net at U6.12 (AINN1): now also C27.1, C29.2, R27.2; no longer J1.9 (Pin_9)
- net at J1.6 (Pin_6): now also R20.1; no longer U6.13 (AINP3)
- net at J1.5 (Pin_5): now also R23.1; no longer U6.14 (AINN3)
- net at J1.3 (Pin_3): now also R17.1; no longer U6.15 (AINN4)
- net at J1.4 (Pin_4): now also R19.1; no longer U6.16 (AINP4)
- net at J1.7 (Pin_7): now also R25.1; no longer U6.17 (AINN2)
- net at J1.8 (Pin_8): now also R24.1; no longer U6.18 (AINP2)
- net at ESP3.3V1.2 (Pin_2), U2.16 (3V3): now also S1.4
- new net: J1.10 (Pin_10), R26.1
- new net: J1.9 (Pin_9), R27.1
- new net N2: C24.1, C26.2, R25.2, U6.17 (AINN2)
- new net N3: C21.1, C23.2, R23.2, U6.14 (AINN3)
- new net N4: C18.1, C20.2, R17.2, U6.15 (AINN4)
- new net P2: C24.2, C25.2, R24.2, U6.18 (AINP2)
- new net P3: C21.2, C22.2, R20.2, U6.13 (AINP3)
- new net P4: C18.2, C19.2, R19.2, U6.16 (AINP4)
Other:
- moved on the sheet: ADC1, C1, C12, C13, C17, DMS1, J1, Q4, R13, R18, R22, U6
